File: hardware/kicad/EcoTwin_Board.kicad_pcb (KiCad board)
At the start: 2 copper layers, 95 x 60 mm, 39 parts, among them J1 USB-C power only, J10 Reed switch, J11 DS18B20 probe, J14 I2C, J15 DevKit right pin row, J16 HX711 input side, J2 IP5306 module, J3 To module B+ / B-, J4 DevKit left pin row, J5 HX711 output side, J6 Load cell cable, J7 E-paper 2.9 in, J9 LED strip, Q1 MMBT3904, SW1 SW_Push, U1 74AHCT1G125

Commit message: Place components
Parts:
- BT1: moved to B.Cu
- moved R1 159.1 mm to (184.0, 116.0)
- moved D1 145.0 mm to (175.0, 110.5)
- moved R2 144.7 mm to (184.0, 119.5)
- moved BZ1 141.2 mm to (176.0, 150.0)
- moved J3 137.1 mm to (167.0, 122.5)
- moved D2 131.0 mm to (175.0, 116.0)
- moved D3 130.6 mm to (181.0, 158.0)
- moved R10 119.1 mm to (160.0, 143.0)
- moved J4 118.7 mm to (161.3, 110.0), turned to -90 degrees
- moved SW1 113.4 mm to (180.0, 135.5)
- moved R9 111.3 mm to (138.0, 143.0)
- moved R11 108.9 mm to (163.5, 143.0)
- moved J1 105.5 mm to (191.5, 117.0), turned to 90 degrees
- moved J14 103.4 mm to (161.0, 151.0)
- moved F1 103.3 mm to (175.0, 106.0)
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